File: first_keyboard_project/first_keyboard_project.kicad_pcb (KiCad board)
At the start: 2 copper layers, 19 parts, among them U1 Arduino_Pro_Micro

Commit message: added first project and prototype
Parts:
- moved D2 19.1 mm to (152.4, 57.1), turned to -90 degrees
- moved D5 19.1 mm to (152.4, 76.2), turned to -90 degrees
- moved D8 19.1 mm to (152.4, 95.2), turned to -90 degrees
- moved D1 19.0 mm to (133.3, 57.1), turned to -90 degrees
- moved D4 19.0 mm to (133.3, 76.2), turned to -90 degrees
- moved D7 19.0 mm to (133.3, 95.2), turned to -90 degrees
- moved D3 19.0 mm to (171.4, 57.1), turned to -90 degrees
- moved D6 19.0 mm to (171.4, 76.2), turned to -90 degrees
- moved D9 19.0 mm to (171.4, 95.2), turned to -90 degrees
Routing:
- net Column 0: track 0.00 -> 108.0 mm
- net Column 1: track 0.00 -> 92.6 mm
- net Column 2: track 0.00 -> 71.6 mm
- net Row 0: track 0.00 -> 71.4 mm
- net Row 1: track 0.00 -> 54.9 mm
- net Row 2: track 0.00 -> 46.0 mm
- net Net-(D8-A): track 0.00 -> 8.30 mm
- net Net-(D7-A): track 0.00 -> 8.30 mm
- net Net-(D5-A): track 0.00 -> 8.30 mm
- net Net-(D2-A): track 0.00 -> 8.30 mm
- net Net-(D4-A): track 0.00 -> 8.30 mm
- net Net-(D1-A): track 0.00 -> 8.30 mm
- net Net-(D9-A): track 0.00 -> 8.30 mm
- net Net-(D6-A): track 0.00 -> 8.30 mm
- net Net-(D3-A): track 0.00 -> 8.30 mm
- added copper zone on B.Cu, net (none)
- added copper zone on F.Cu, net (none)
Other:
- board outline added: 86.8 x 65.2 mm
